Commit message: add MoveIt Servo teleop simulation support

File: ros2_ws/src/redburi_description/urdf/arm.urdf.xacro (robot description, xacro)
@@ -9,7 +9,7 @@
   <xacro:property name="link1_len" value="0.25"/>
   <xacro:property name="link2_len" value="0.25"/>
-  <xacro:property name="link3_len" value="0.25"/>
-  <xacro:property name="link4_len" value="0.2"/>
-  <xacro:property name="link5_len" value="0.1"/>
+  <xacro:property name="link3_len" value="0.257"/>
+  <xacro:property name="link4_len" value="0.214"/>
+  <xacro:property name="link5_len" value="0.052"/>
   <xacro:property name="link6_len" value="0.25"/>
   <xacro:property name="gripper_w" value="0.03"/>
@@ -52,5 +52,5 @@
       <!-- arm body -->
       <visual>
-        <origin xyz="0 0 ${link_len/2.0}" rpy="0 0 0"/>
+        <origin xyz="0 0 ${float(link_len) / 2.0}" rpy="0 0 0"/>
         <geometry>
           <box size="${link_w} ${link_h} ${link_len}"/>
@@ -59,5 +59,5 @@
       </visual>
       <collision>
-        <origin xyz="0 0 ${link_len/2.0}" rpy="0 0 0"/>
+        <origin xyz="0 0 ${float(link_len) / 2.0}" rpy="0 0 0"/>
         <geometry>
           <box size="${link_w} ${link_h} ${link_len}"/>
@@ -71,5 +71,5 @@
       <!-- arm body -->
       <visual>
-        <origin xyz="0 0 ${link_len/2.0}" rpy="0 0 0"/>
+        <origin xyz="0 0 ${float(link_len) / 2.0}" rpy="0 0 0"/>
         <geometry>
           <box size="${link_w} ${link_h} ${link_len}"/>
@@ -78,5 +78,5 @@
       </visual>
       <collision>
-        <origin xyz="0 0 ${link_len/2.0}" rpy="0 0 0"/>
+        <origin xyz="0 0 ${float(link_len) / 2.0}" rpy="0 0 0"/>
         <geometry>
           <box size="${link_w} ${link_h} ${link_len}"/>
@@ -99,5 +99,5 @@
       <!-- arm body -->
       <visual>
-        <origin xyz="0 0 ${link_len/2.0}" rpy="0 0 0"/>
+        <origin xyz="0 0 ${float(link_len) / 2.0}" rpy="0 0 0"/>
         <geometry>
           <box size="${link_w} ${link_h} ${link_len}"/>
@@ -112,5 +112,5 @@
       </collision>
       <collision>
-        <origin xyz="0 0 ${link_len/2.0}" rpy="0 0 0"/>
+        <origin xyz="0 0 ${float(link_len) / 2.0}" rpy="0 0 0"/>
         <geometry>
           <box size="${link_w} ${link_h} ${link_len}"/>
